File: PCB/apex-alpha-ii.sch (EAGLE design)
At the start: 36 parts, among them IC1 CC430F5135, IC2 TPS61200, X2 SMA-142-0711-871/876, Y1 26MHz

Commit message: Flipped battery - still AAA
Parts:
- X2: value SMA-142-0711-871/876 -> SMA-142-0701-801/806; device con-coax:SMA-142-0711-871/876 -> !danielparts:SMA-142-0701-801/806; MPN (none) -> 142-0701-801; OC_FARNELL (none) -> 1608592; OC_NEWARK (none) -> 90F2624
Changed lines of the file:
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@@
 <layer number="19" name="Unrouted" color="6" fill="1" visible="no" active="no"/>
 <layer number="20" name="Dimension" color="15" fill="1" visible="no" active="no"/>
-<layer number="21" name="tPlace" color="7" fill="1" visible="no" active="no"/>
-<layer number="22" name="bPlace" color="7" fill="1" visible="no" active="no"/>
+<layer number="21" name="tPlace" color="16" fill="1" visible="no" active="no"/>
+<layer number="22" name="bPlace" color="14" fill="1" visible="no" active="no"/>
 <layer number="23" name="tOrigins" color="15" fill="1" visible="no" active="no"/>
 <layer number="24" name="bOrigins" color="15" fill="1" visible="no" active="no"/>
@@
 <layer number="49" name="Reference" color="7" fill="1" visible="no" active="no"/>
 <layer number="50" name="dxf" color="7" fill="1" visible="no" active="no"/>
-<layer number="51" name="tDocu" color="7" fill="1" visible="no" active="no"/>
+<layer number="51" name="tDocu" color="6" fill="1" visible="no" active="no"/>
 <layer number="52" name="bDocu" color="7" fill="1" visible="no" active="no"/>
 <layer number="53" name="tGND_GNDA" color="7" fill="9" visible="no" active="no"/>
@@
 <part name="GND9" library="apex" deviceset="GND" device=""/>
 <part name="P+3" library="apex" deviceset="VCC" device=""/>
-<part name="X2" library="con-coax" deviceset="SMA-" device="142-0711-871/876" value=""/>
+<part name="X2" library="!danielparts" deviceset="SMA-" device="142-0701-801/806" value="">
+<attribute name="MPN" value="142-0701-801"/>
+<attribute name="OC_FARNELL" value="1608592"/>
+<attribute name="OC_NEWARK" value="90F2624"/>
+</part>
 <part name="GND10" library="apex" deviceset="GND" device=""/>
 <part name="GND11" library="apex" deviceset="GND" device=""/>
