File: PCB/apex-alpha-ii.brd (EAGLE design)
At the start: 19.2 x 60.5 mm, 31 parts, among them IC1 CC430F5135, Y1 26MHz

Commit message: Final PCB layout
Parts:
- removed CR123A: (no value), apex:SMD-BATTERY-HOLDER-CR123A
- removed JP1: APEXHAB-LOGO_APEXHAB-SMALL, apex:APEXHAB-LOGO-SMALL
- removed VREG: TLV70019, !danielparts:SC70-5L
- added AAA: (no value), apex:THROUGH-HOLE-BATTERY-HOLDER-AAA
- added C1: 1uF, apex:0402-CAP
- added C19: 4.7uF, apex:0805
- added C6: 100nF, apex:0402-CAP
- added IC2: TPS61200, texas:S-PDSO-N10
- added NR3015: 2.2uH, apex:NR3015
- added R1: 560k, apex:R0402
- added R2: 200k, apex:R0402
- added TP3: PTR1B1,27, testpad:B1,27
- added U$4: APEX, !danielparts:APEXHAB-LOGO-SMALL
- added U$5: (no value), !danielparts:APEXHAB-LOGO-SMALL
- C10: value 10uF -> 1uF
- C2, C3: value 1uF -> 10uF; device apex:0402-CAP -> apex:0805
- C9: value 10uF -> 100nF
- TP1, TP2: value PTR1B2,54 -> PTR1B1,27; device testpad:B2,54 -> testpad:B1,27
- U$3: device apex:CHIPLED_0805 -> apex:R0402
- moved R4 74.7 mm to (11.9, 18.0), turned to 90 degrees
- moved R3 69.2 mm to (8.89, 13.0), turned to 90 degrees
- moved C8 65.5 mm to (1.52, 19.1), turned to 90 degrees
- moved C16 65.0 mm to (4.83, 6.86), turned to 270 degrees
- moved C5 64.0 mm to (11.9, 20.6), turned to 270 degrees
- moved C7 63.4 mm to (5.59, 24.8), turned to 270 degrees
- moved C18 63.1 mm to (11.0, 34.5)
- moved C4 63.0 mm to (11.9, 15.5), turned to 270 degrees
- moved Y1 62.6 mm to (2.29, 8.64), turned to 270 degrees
- moved C17 61.3 mm to (1.52, 13.0), turned to 270 degrees
- moved C14 59.4 mm to (10.4, 13.0), turned to 270 degrees
- moved C2 59.2 mm to (2.92, 29.6), turned to 90 degrees
- moved C15 58.1 mm to (4.83, 13.0), turned to 270 degrees
- moved F1 55.8 mm to (6.10, 9.91)
- moved IC1 55.1 mm to (6.60, 19.1)
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Connections:
- new net N$1: AAA.+V, C2.2, IC2.5, IC2.6, IC2.7, IC2.8, NR3015.P$1
- new net N$4: IC2.10, R1.1, R2.2
- new net N$5: C1.1, IC2.1
- new net VEE: C11.1, C12.1, C13.1, C14.1, C15.1, IC1.27, IC1.28, IC1.31, IC1.32, IC1.34, U$2.2
- net GND: now also AAA.GND, C1.2, C19.2, C6.2, IC2.4, IC2.9, IC2.PP, IC2.PP@1, IC2.PP@2, R2.1, U$3.1; no longer CR123A.GND, U$3.C, VREG.2
- net N$15: now also U$3.2; no longer U$3.A
- net N$3: now also IC2.3, NR3015.P$2; no longer C2.2, CR123A.+V, VREG.1, VREG.3
- net VCC: now also C19.1, C6.1, IC2.2, R1.2, TP3.TP; no longer C11.1, C12.1, C13.1, C14.1, C15.1, IC1.27, IC1.28, IC1.31, IC1.32, IC1.34, U$2.2, VREG.5
Routing:
- net VCC: track 0.00 -> 56.4 mm, vias 0 -> 3
- net N$1: track 0.00 -> 31.4 mm, vias 0 -> 2
- net GPSRX: track 0.00 -> 23.0 mm, vias 0 -> 2
- net GPSTX: track 0.00 -> 22.1 mm, vias 0 -> 2
- net VEE: track 0.00 -> 19.3 mm
- net N$12: track 0.00 -> 11.4 mm, vias 0 -> 2
- net N$14: track 0.00 -> 10.9 mm, vias 0 -> 2
- net N$11: track 0.00 -> 10.1 mm, vias 0 -> 2
- net N$13: track 0.00 -> 9.90 mm
- net N$7: track 0.00 -> 8.49 mm
- net N$8: track 0.00 -> 5.89 mm
- net N$4: track 0.00 -> 3.50 mm
- net GND: track 0.00 -> 3.02 mm, vias 0 -> 46
- net N$3: track 0.00 -> 2.66 mm
- net N$9: track 0.00 -> 2.40 mm
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- added copper zone on layer 1, net GND
- added copper zone on layer 16, net GND
- added copper zone on layer 1, net N$1
- added copper zone on layer 1, net N$2
- added copper zone on layer 1, net N$6
Other:
- board size 19.2 x 60.5 mm -> 13.1 x 62.2 mm
- board text added: "ALPHA"
- board text added: "APEX"
- board text added: "AUG 2013"
- board text added: "CC430"
- board text added: "DANIEL"
- board text added: "Mk II"
- board text added: "SAUL"
- board text added: "STATUS"
- board text added: "VCC"

Commit message: Generated gerbers
Parts:
- moved U$4 26.1 mm to (-0.76, 50.4)
Other:
- board text added: "ALPHA II"
- board text added: "AUGUST 2013"
- board text added: "DANIEL SAUL"
- board text removed: "ALPHA"
- board text removed: "APEX"
- board text removed: "AUG 2013"
- board text removed: "DANIEL"
- board text removed: "Mk II"
- board text removed: "SAUL"
Changed lines of the file:
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@@
 <setting verticaltext="up"/>
 </settings>
-<grid distance="0.005" unitdist="inch" unit="mm" style="dots" multiple="1" display="yes" altdistance="0.001" altunitdist="inch" altunit="inch"/>
+<grid distance="0.01" unitdist="inch" unit="inch" style="dots" multiple="1" display="yes" altdistance="0.001" altunitdist="inch" altunit="inch"/>
 <layers>
 <layer number="1" name="Top" color="4" fill="1" visible="yes" active="yes"/>
@@
 <wire x1="1.744121875" y1="0" x2="11.387878125" y2="0" width="0" layer="20"/>
 <wire x1="11.387878125" y1="0" x2="13.132" y2="1.744121875" width="0" layer="20" curve="90"/>
-<text x="7.366" y="61.214" size="1.778" layer="21" font="vector" ratio="15" rot="R180">APEX</text>
-<text x="9.017" y="58.42" size="1.778" layer="21" font="vector" ratio="15" rot="R180">ALPHA</text>
-<text x="0.762" y="53.848" size="1.778" layer="21" font="vector" ratio="15">Mk II</text>
-<text x="11.049" y="59.436" size="1.778" layer="22" font="vector" ratio="15" rot="MR0">DANIEL</text>
-<text x="9.525" y="57.277" size="1.778" layer="22" font="vector" ratio="15" rot="MR0">SAUL</text>
-<text x="11.303" y="54.864" size="1.27" layer="22" font="vector" ratio="15" rot="MR0">AUG 2013</text>
+<text x="12.446" y="58.7502" size="1.778" layer="22" font="vector" ratio="15" rot="MR0">ALPHA II</text>
+<text x="11.4554" y="56.7436" size="1.016" layer="22" font="vector" ratio="15" rot="MR0">DANIEL SAUL</text>
 <text x="8.763" y="35.179" size="0.6096" layer="21" font="vector" ratio="15" rot="R180">VCC</text>
 <text x="7.62" y="14.859" size="0.6096" layer="21" font="vector" ratio="15" rot="R180">CC430</text>
 <text x="11.684" y="25.146" size="0.6096" layer="21" font="vector" ratio="15" rot="R180">STATUS</text>
+<text x="11.6332" y="55.2196" size="1.016" layer="22" font="vector" ratio="15" rot="MR0">AUGUST 2013</text>
 </plain>
 <attributes>
@@
 <element name="C18" library="apex" package="0402-CAP" value="100nF" x="11.049" y="34.544"/>
 <element name="C19" library="apex" package="0805" value="4.7uF" x="10.795" y="36.195"/>
-<element name="U$4" library="!danielparts" package="APEXHAB-LOGO-SMALL" value="APEX" x="1.143" y="24.384"/>
+<element name="U$4" library="!danielparts" package="APEXHAB-LOGO-SMALL" value="APEX" x="-0.762" y="50.419"/>
 <element name="U$5" library="!danielparts" package="APEXHAB-LOGO-SMALL" value="" x="11.684" y="24.384" rot="MR0"/>
 <element name="TP3" library="testpad" package="B1,27" value="PTR1B1,27" x="7.874" y="36.068">
@@
 </signal>
 </signals>
-<errors>
-</errors>
 </board>
 </drawing>
